File: EE_156_HalloweenPCB.kicad_pcb (KiCad board)
At the start: 2 copper layers, 0 parts

Commit message: add adafruit library
Other:
- board outline added: 115.5 x 75.1 mm
Changed lines of the file:
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@@
   )
   (net 0 "")
+  (gr_rect (start 142.9512 78.994) (end 258.4958 154.0764)
+    (stroke (width 0.1) (type default)) (fill none) (layer "Edge.Cuts"))
 )
