File: EE_156_HalloweenPCB.kicad_sch (KiCad schematic)
At the start: 46 parts, among them J1 Conn_01x04_Male, J2 B2B-PH-SM4-TB, J3 Conn_01x04_Male, J4 Conn_01x04_Male, J5 Conn_01x04_Male, J6 Conn_01x04_Male, J7 USB_C_Receptacle_USB2.0, Q1 DMG341, U1 MCP73831T-2ACI/OT, U2 ATSAMD21G18A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

Commit message: add adafruit library
Parts:
- U3: footprint Trinket M0 rev D:SOT23-5 -> EE156_HalloweenPCB:SOT23-5; Datasheet Link (none) -> https://www.diodes.com/assets/Datasheets/AP2112.pdf; DigiKey Part Number (none) -> AP2112K-3.3TRG1DICT-ND
Connections:
- no-connect marks 1 -> 8
Changed lines of the file:
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@@
   )
   (no_connect (at 138.43 92.71))
+  (no_connect (at 320.04 106.68))
+  (no_connect (at 320.04 76.2))
+  (no_connect (at 320.04 93.98))
+  (no_connect (at 328.2188 84.582))
+  (no_connect (at 320.04 73.66))
+  (no_connect (at 320.04 78.74))
+  (no_connect (at 320.04 119.38))
   (wire (pts (xy 80.01 63.5) (xy 77.47 63.5))
     (stroke (width 0) (type default))
@@
       (effects (font (size 1.0668 1.0668)) (justify left bottom))
     )
-    (property "Footprint" "Trinket M0 rev D:SOT23-5" (at 128.27 90.17 0)
+    (property "Footprint" "EE156_HalloweenPCB:SOT23-5" (at 128.27 90.17 0)
       (effects (font (size 1.27 1.27)) hide)
     )
@@
       (effects (font (size 1.27 1.27)) hide)
     )
+    (property "DigiKey Part Number" "AP2112K-3.3TRG1DICT-ND" (at 128.27 90.17 0)
+      (effects (font (size 1.27 1.27)) hide)
+    )
+    (property "Datasheet Link" "https://www.diodes.com/assets/Datasheets/AP2112.pdf" (at 128.27 90.17 0)
+      (effects (font (size 1.27 1.27)) hide)
+    )
+    (property "Tolerance" "" (at 128.27 90.17 0)
+      (effects (font (size 1.27 1.27)))
+    )
+    (property "Power Rating" "" (at 128.27 90.17 0)
+      (effects (font (size 1.27 1.27)))
+    )
     (pin "1")
